Commit message: 1may

File: ur_ws_new/src/ur_robot_driver/ur_description/urdf/ur_macro.xacro (robot description, xacro)
@@ -337,4 +337,39 @@
       <child link="${prefix}tool0"/>
     </joint>
+    <joint name="${prefix}tool0_to_gripper" type="fixed">
+  		<parent link="${prefix}tool0"/>
+  		<child link="${prefix}gripper_link"/>
+  		<origin xyz="0 0 0" rpy="0 0 0"/>
+		</joint>
+    <joint name="${prefix}gripper_link_to_tip" type="fixed">
+  		<parent link="${prefix}gripper_link"/>
+  		<child link="${prefix}gripper_tip"/>
+  		<origin xyz="0 0 0.23" rpy="0 0 0"/> <!-- Match the box length -->
+		</joint>
+    <!-- Gripper geometry attached to tool0 -->
+<link name="${prefix}gripper_link">
+  <visual>
+    <origin xyz="0 0 0.0" rpy="0 0 0"/> <!-- adjust offset as needed -->
+    <geometry>
+      <box size="0.07 0.07 0.19"/> <!-- dimensions of your gripper -->
+    </geometry>
+    <material name="gray">
+      <color rgba="0.5 0.5 0.5 1.0"/>
+    </material>
+  </visual>
+  <collision>
+    <origin xyz="0 0 0.0" rpy="0 0 0"/>
+    <geometry>
+      <box size="0.05 0.05 0.19"/>
+    </geometry>
+  </collision>
+  <inertial>
+    <mass value="0.5"/>
+    <origin xyz="0 0 0.1" rpy="0 0 0"/>
+    <inertia ixx="0.001" ixy="0.0" ixz="0.0" iyy="0.001" iyz="0.0" izz="0.001"/>
+  </inertial>
+</link>
+<!-- Gripper tip frame -->
+<link name="${prefix}gripper_tip"/>
   </xacro:macro>
 </robot>

Commit message: 5may

File: ur_ws_new/src/ur_robot_driver/ur_description/urdf/ur_macro.xacro (robot description, xacro)
@@ -340,15 +340,15 @@
   		<parent link="${prefix}tool0"/>
   		<child link="${prefix}gripper_link"/>
-  		<origin xyz="0 0 0" rpy="0 0 0"/>
+  		<origin xyz="0 0 0.01" rpy="0 0 0"/>
 		</joint>
     <joint name="${prefix}gripper_link_to_tip" type="fixed">
   		<parent link="${prefix}gripper_link"/>
   		<child link="${prefix}gripper_tip"/>
-  		<origin xyz="0 0 0.23" rpy="0 0 0"/> <!-- Match the box length -->
+  		<origin xyz="0 0 0.205" rpy="0 0 0"/> <!-- Match the box length -->
 		</joint>
     <!-- Gripper geometry attached to tool0 -->
 <link name="${prefix}gripper_link">
   <visual>
-    <origin xyz="0 0 0.0" rpy="0 0 0"/> <!-- adjust offset as needed -->
+    <origin xyz="0 0 0.1" rpy="0 0 0"/> <!-- adjust offset as needed -->
     <geometry>
       <box size="0.07 0.07 0.19"/> <!-- dimensions of your gripper -->

Commit message: before jetson change

File: ur_ws_new/src/ur_robot_driver/ur_description/urdf/ur_macro.xacro (robot description, xacro)
@@ -337,4 +337,10 @@
       <child link="${prefix}tool0"/>
     </joint>
+      <link name="zed2_left_camera_frame"/>
+  <joint name="tool0_to_zed2_left_camera_frame" type="fixed">
+    <parent link="tool0"/>
+    <child link="zed2_left_camera_frame"/>
+    <origin xyz="-0.06 -0.14 0.06" rpy="0 0 0"/>
+  </joint>
     <joint name="${prefix}tool0_to_gripper" type="fixed">
   		<parent link="${prefix}tool0"/>

Commit message: 21may

File: ur_ws_new/src/ur_robot_driver/ur_description/urdf/ur_macro.xacro (robot description, xacro)
@@ -351,5 +351,5 @@
   		<parent link="${prefix}gripper_link"/>
   		<child link="${prefix}gripper_tip"/>
-  		<origin xyz="0 0 0.205" rpy="0 0 0"/> <!-- Match the box length -->
+  		<origin xyz="0 0 0.225" rpy="0 0 0"/> <!-- Match the box length -->
 		</joint>
     <!-- Gripper geometry attached to tool0 -->
