Commit message: 21Dec

File: ur_ws_new/src/universal_robot/urdf/ur_macro.xacro (robot description, xacro)
@@ -451,7 +451,7 @@
     <link name="tool0_to_camera_mount_link">
   <visual>
-    <origin xyz="0.045 0.04 -0.005" rpy="0 0 3.14159"/>
+    <origin xyz="0.0 0.0 -0.032" rpy="0 0 3.14159"/>
     <geometry>
-      <mesh filename="package://ur_description/meshes/ur10e/visual/mount.stl" scale="0.001 0.001 0.001"/>
+      <mesh filename="package://ur_description/meshes/ur10e/visual/top_zed_homut.stl" scale="0.001 0.001 0.001"/>
     </geometry>
     <material name="silver">
@@ -462,5 +462,5 @@
     <origin xyz="0.045 0.04 -0.005" rpy="0 0 3.14159"/>
     <geometry>
-      <mesh filename="package://ur_description/meshes/ur10e/visual/mount.stl" scale="0.001 0.001 0.001"/>
+      <mesh filename="package://ur_description/meshes/ur10e/visual/top_zed_homut.stl" scale="0.001 0.001 0.001"/>
     </geometry>
   </collision>
@@ -501,5 +501,5 @@
     <parent link="tool0"/>
     <child link="zed2_left_camera_frame"/>
-    <origin xyz="-0.037 -0.131 0.038" rpy="0 0 -0.174"/>   <!-- CHANGE -->
+    <origin xyz="-0.048 -0.156 -0.005" rpy="0 0 -0.174"/>   <!-- CHANGE -->
   </joint>
     <joint name="${tf_prefix}gripper_link_to_tip" type="fixed">

Commit message: livox integration to main

File: ur_ws_new/src/universal_robot/urdf/ur_macro.xacro (robot description, xacro)
@@ -8,5 +8,5 @@
     This file models the base kinematic chain of a UR robot, which then gets
     parameterised by various configuration files to convert it into a UR3(e),
-    UR5(e), UR10(e) or UR16e, etc.
+    UR5(e), UR10(e) or UR16e.
     NOTE the default kinematic parameters (i.e., link lengths, frame locations,
     offsets, etc) do not correspond to any particular robot. They are defaults
@@ -46,13 +46,9 @@
   <xacro:include filename="$(find delto_description)/urdf/delto_gripper_3f.xacro"/>
   <xacro:macro name="ur_robot" params="
-    name
-    tf_prefix
-    parent
-    *origin
+    prefix
     joint_limits_parameters_file
     kinematics_parameters_file
     physical_parameters_file
     visual_parameters_file
-    generate_ros2_control_tag:=true
     transmission_hw_interface:=hardware_interface/PositionJointInterface
     safety_limits:=false
@@ -61,29 +57,5 @@
     use_fake_hardware:=false
     fake_sensor_commands:=false
-    sim_gazebo:=false
-    sim_ignition:=false
-    headless_mode:=false
-    initial_positions:=${dict(shoulder_pan_joint=0.0,shoulder_lift_joint=-1.57,elbow_joint=0.0,wrist_1_joint=-1.57,wrist_2_joint=0.0,wrist_3_joint=0.0)}
-    use_tool_communication:=false
-    tool_voltage:=0
-    tool_parity:=0
-    tool_baud_rate:=115200
-    tool_stop_bits:=1
-    tool_rx_idle_chars:=1.5
-    tool_tx_idle_chars:=3.5
-    tool_device_name:=/tmp/ttyUR
-    tool_tcp_port:=54321
-    robot_ip:=0.0.0.0
-    script_filename:=to_be_filled_by_ur_robot_driver
-    output_recipe_filename:=to_be_filled_by_ur_robot_driver
-    input_recipe_filename:=to_be_filled_by_ur_robot_driver
-    reverse_port:=50001
-    script_sender_port:=50002
-    reverse_ip:=0.0.0.0
-    script_command_port:=50004
-    trajectory_port:=50003
-    non_blocking_read:=true
-    keep_alive_count:=2"
-    >
+    initial_positions:=${dict(shoulder_pan_joint=0.0,shoulder_lift_joint=-1.57,elbow_joint=0.0,wrist_1_joint=-1.57,wrist_2_joint=0.0,wrist_3_joint=0.0)}">
     <!-- Load configuration data from the provided .yaml files -->
     <xacro:read_model_data
@@ -91,58 +63,43 @@
       kinematics_parameters_file="${kinematics_parameters_file}"
       physical_parameters_file="${physical_parameters_file}"
-      visual_parameters_file="${visual_parameters_file}"
-      force_abs_paths="${sim_gazebo or sim_ignition}"/>
-    <xacro:if value="${generate_ros2_control_tag}">
-      <!-- ros2 control include -->
-      <xacro:include filename="$(find ur_description)/urdf/ur.ros2_control.xacro" />
-      <!-- ros2 control instance -->
-      <xacro:ur_ros2_control
-        name="${name}"
-        use_fake_hardware="${use_fake_hardware}"
-        initial_positions="${initial_positions}"
-        fake_sensor_commands="${fake_sensor_commands}"
-        headless_mode="${headless_mode}"
-        sim_gazebo="${sim_gazebo}"
-        sim_ignition="${sim_ignition}"
-        script_filename="${script_filename}"
-        output_recipe_filename="${output_recipe_filename}"
-        input_recipe_filename="${input_recipe_filename}"
-        tf_prefix="${tf_prefix}"
-        hash_kinematics="${kinematics_hash}"
-        robot_ip="${robot_ip}"
-        use_tool_communication="${use_tool_communication}"
-        tool_voltage="${tool_voltage}"
-        tool_parity="${tool_parity}"
-        tool_baud_rate="${tool_baud_rate}"
-        tool_stop_bits="${tool_stop_bits}"
-        tool_rx_idle_chars="${tool_rx_idle_chars}"
-        tool_tx_idle_chars="${tool_tx_idle_chars}"
-        tool_device_name="${tool_device_name}"
-        tool_tcp_port="${tool_tcp_port}"
-        reverse_port="${reverse_port}"
-        script_sender_port="${script_sender_port}"
-        reverse_ip="${reverse_ip}"
-        script_command_port="${script_command_port}"
-        trajectory_port="${trajectory_port}"
-        non_blocking_read="${non_blocking_read}"
-        keep_alive_count="${keep_alive_count}"
-        />
-    </xacro:if>
+      visual_parameters_file="${visual_parameters_file}"/>
+    <!-- Data files required by the UR driver -->
+    <xacro:arg name="script_filename" default="$(find ur_robot_driver)/resources/ros_control.urscript"/>
+    <xacro:arg name="output_recipe_filename" default="$(find ur_robot_driver)/resources/rtde_output_recipe.txt"/>
+    <xacro:arg name="input_recipe_filename" default="$(find ur_robot_driver)/resources/rtde_input_recipe.txt"/>
+    <xacro:arg name="robot_ip" default="10.0.1.186"/>
+    <!-- ros2 control include -->
+    <xacro:include filename="$(find ur_description)/urdf/ur.ros2_control.xacro" />
+    <!-- ros2 control instance -->
+    <xacro:ur_ros2_control
+      name="URPositionHardwareInterface" prefix="${prefix}"
+      use_fake_hardware="$(arg use_fake_hardware)"
+      initial_positions="${initial_positions}"
+      fake_sensor_commands="$(arg fake_sensor_commands)"
+      script_filename="$(arg script_filename)"
+      output_recipe_filename="$(arg output_recipe_filename)"
+      input_recipe_filename="$(arg input_recipe_filename)"
+      tf_prefix=""
+      hash_kinematics="${kinematics_hash}"
+      robot_ip="$(arg robot_ip)" />
     <!-- Add URDF transmission elements (for ros_control) -->
     <!--<xacro:ur_arm_transmission prefix="${prefix}" hw_interface="${transmission_hw_interface}" />-->
     <!-- Placeholder for ros2_control transmission which don't yet exist -->
     <!-- links -  main serial chain -->
-    <link name="${tf_prefix}base_link"/>
-    <link name="${tf_prefix}base_link_inertia">
+    <link name="${prefix}base_link"/>
+    <link name="${prefix}base_link_inertia">
       <visual>
         <origin xyz="0 0 0" rpy="0 0 ${pi}"/>
         <geometry>
-          <xacro:get_mesh name="base" type="visual"/>
-        </geometry>
+          <mesh filename="${base_visual_mesh}"/>
+        </geometry>
+        <material name="${base_visual_material_name}">
+          <color rgba="${base_visual_material_color}"/>
+        </material>
       </visual>
       <collision>
         <origin xyz="0 0 0" rpy="0 0 ${pi}"/>
         <geometry>
-          <xacro:get_mesh name="base" type="collision"/>
+          <mesh filename="${base_collision_mesh}"/>
         </geometry>
       </collision>
@@ -151,178 +108,128 @@
       </xacro:cylinder_inertial>
     </link>
-    <link name="${tf_prefix}shoulder_link">
+    <link name="${prefix}shoulder_link">
       <visual>
         <origin xyz="0 0 0" rpy="0 0 ${pi}"/>
         <geometry>
-          <xacro:get_mesh name="shoulder" type="visual"/>
-        </geometry>
+          <mesh filename="${shoulder_visual_mesh}"/>
+        </geometry>
+        <material name="${shoulder_visual_material_name}">
+          <color rgba="${shoulder_visual_material_color}"/>
+        </material>
       </visual>
       <collision>
         <origin xyz="0 0 0" rpy="0 0 ${pi}"/>
         <geometry>
-          <xacro:get_mesh name="shoulder" type="collision"/>
-        </geometry>
-      </collision>
-      <inertial>
-        <mass value="${shoulder_mass}"/>
-        <origin rpy="${shoulder_inertia_rotation}" xyz="${shoulder_cog}"/>
-        <inertia
-            ixx="${shoulder_inertia_ixx}"
-            ixy="${shoulder_inertia_ixy}"
-            ixz="${shoulder_inertia_ixz}"
-            iyy="${shoulder_inertia_iyy}"
-            iyz="${shoulder_inertia_iyz}"
-            izz="${shoulder_inertia_izz}"
-        />
-      </inertial>    </link>
-    <link name="${tf_prefix}upper_arm_link">
+          <mesh filename="${shoulder_collision_mesh}"/>
+        </geometry>
+      </collision>
+      <xacro:cylinder_inertial radius="${shoulder_inertia_radius}" length="${shoulder_inertia_length}" mass="${shoulder_mass}">
+        <origin xyz="0 0 0" rpy="0 0 0" />
+      </xacro:cylinder_inertial>
+    </link>
+    <link name="${prefix}upper_arm_link">
       <visual>
         <origin xyz="0 0 ${shoulder_offset}" rpy="${pi/2} 0 ${-pi/2}"/>
         <geometry>
-          <xacro:get_mesh name="upper_arm" type="visual"/>
-        </geometry>
+          <mesh filename="${upper_arm_visual_mesh}"/>
+        </geometry>
+        <material name="${upper_arm_visual_material_name}">
+          <color rgba="${upper_arm_visual_material_color}"/>
+        </material>
       </visual>
       <collision>
         <origin xyz="0 0 ${shoulder_offset}" rpy="${pi/2} 0 ${-pi/2}"/>
         <geometry>
-          <xacro:get_mesh name="upper_arm" type="collision"/>
-        </geometry>
-      </collision>
-      <inertial>
-        <mass value="${upper_arm_mass}"/>
-        <origin rpy="${upper_arm_inertia_rotation}" xyz="${upper_arm_cog}"/>
-        <inertia
-            ixx="${upper_arm_inertia_ixx}"
-            ixy="${upper_arm_inertia_ixy}"
-            ixz="${upper_arm_inertia_ixz}"
-            iyy="${upper_arm_inertia_iyy}"
-            iyz="${upper_arm_inertia_iyz}"
-            izz="${upper_arm_inertia_izz}"
-        />
-      </inertial>
-    </link>
-    <link name="${tf_prefix}forearm_link">
+          <mesh filename="${upper_arm_collision_mesh}"/>
+        </geometry>
+      </collision>
+      <xacro:cylinder_inertial radius="${upperarm_inertia_radius}" length="${upperarm_inertia_length}" mass="${upper_arm_mass}">
+        <origin xyz="${-0.5 * upperarm_inertia_length} 0.0 ${upper_arm_inertia_offset}" rpy="0 ${pi/2} 0" />
+      </xacro:cylinder_inertial>
+    </link>
+    <link name="${prefix}forearm_link">
       <visual>
         <origin xyz="0 0 ${elbow_offset}" rpy="${pi/2} 0 ${-pi/2}"/>
         <geometry>
-          <xacro:get_mesh name="forearm" type="visual"/>
-        </geometry>
+          <mesh filename="${forearm_visual_mesh}"/>
+        </geometry>
+        <material name="${forearm_visual_material_name}">
+          <color rgba="${forearm_visual_material_color}"/>
+        </material>
       </visual>
       <collision>
         <origin xyz="0 0 ${elbow_offset}" rpy="${pi/2} 0 ${-pi/2}"/>
         <geometry>
-          <xacro:get_mesh name="forearm" type="collision"/>
-        </geometry>
-      </collision>
-      <inertial>
-        <mass value="${forearm_mass}"/>
-        <origin rpy="${forearm_inertia_rotation}" xyz="${forearm_cog}"/>
-        <inertia
-            ixx="${forearm_inertia_ixx}"
-            ixy="${forearm_inertia_ixy}"
-            ixz="${forearm_inertia_ixz}"
-            iyy="${forearm_inertia_iyy}"
-            iyz="${forearm_inertia_iyz}"
-            izz="${forearm_inertia_izz}"
-        />
-      </inertial>
-    </link>
-    <link name="${tf_prefix}wrist_1_link">
-	  <xacro:get_visual_params name="wrist_1" type="visual_offset"/>
-      <visual>
-      	<origin xyz="0 0 ${visual_params}" rpy="${pi/2} 0 0"/>
-        <geometry>
-          <xacro:get_mesh name="wrist_1" type="visual"/>
-        </geometry>
-      </visual>
-      <collision>
-        <origin xyz="0 0 ${visual_params}" rpy="${pi/2} 0 0"/>
-        <geometry>
-          <xacro:get_mesh name="wrist_1" type="collision"/>
-        </geometry>
-      </collision>
-      <inertial>
-        <mass value="${wrist_1_mass}"/>
-        <origin rpy="${wrist_1_inertia_rotation}" xyz="${wrist_1_cog}"/>
-        <inertia
-            ixx="${wrist_1_inertia_ixx}"
-            ixy="${wrist_1_inertia_ixy}"
-            ixz="${wrist_1_inertia_ixz}"
-            iyy="${wrist_1_inertia_iyy}"
-            iyz="${wrist_1_inertia_iyz}"
-            izz="${wrist_1_inertia_izz}"
-        />
-      </inertial>
-    </link>
-    <link name="${tf_prefix}wrist_2_link">
-          <xacro:get_visual_params name="wrist_2" type="visual_offset"/>
-      <visual>
-        <origin xyz="0 0 ${visual_params}" rpy="0 0 0"/>
-        <geometry>
-          <xacro:get_mesh name="wrist_2" type="visual"/>
-        </geometry>
-      </visual>
-      <collision>
-        <origin xyz="0 0 ${visual_params}" rpy="0 0 0"/>
-        <geometry>
-          <xacro:get_mesh name="wrist_2" type="collision"/>
-        </geometry>
-      </collision>
-      <inertial>
-        <mass value="${wrist_2_mass}"/>
-        <origin rpy="${wrist_2_inertia_rotation}" xyz="${wrist_2_cog}"/>
-        <inertia
-            ixx="${wrist_2_inertia_ixx}"
-            ixy="${wrist_2_inertia_ixy}"
-            ixz="${wrist_2_inertia_ixz}"
-            iyy="${wrist_2_inertia_iyy}"
-            iyz="${wrist_2_inertia_iyz}"
-            izz="${wrist_2_inertia_izz}"
-        />
-      </inertial>
-    </link>
-    <link name="${tf_prefix}wrist_3_link">
-      <!-- TODO: remove this once all wrist_3 meshes have the visual_offset_xyz tag -->
-      <xacro:get_visual_params name="wrist_3" type="visual_offset_xyz"/>
-      <xacro:property name="mesh_offset" value="${visual_params}" scope="parent"/>
-      <xacro:if value="${visual_params == ''}">
-        <xacro:get_visual_params name="wrist_3" type="visual_offset"/>
-        <xacro:property name="mesh_offset" value="0 0 ${visual_params}" scope="parent"/>
-      </xacro:if>
-      <visual>
-        <origin xyz="${mesh_offset}" rpy="${pi/2} 0 0"/>
-        <geometry>
-          <xacro:get_mesh name="wrist_3" type="visual"/>
-        </geometry>
-      </visual>
-      <collision>
-        <origin xyz="${mesh_offset}" rpy="${pi/2} 0 0"/>
-        <geometry>
-          <xacro:get_mesh name="wrist_3" type="collision"/>
-        </geometry>
-      </collision>
-      <inertial>
-        <mass value="${wrist_3_mass}"/>
-        <origin rpy="${wrist_3_inertia_rotation}" xyz="${wrist_3_cog}"/>
-        <inertia
-            ixx="${wrist_3_inertia_ixx}"
-            ixy="${wrist_3_inertia_ixy}"
-            ixz="${wrist_3_inertia_ixz}"
-            iyy="${wrist_3_inertia_iyy}"
-            iyz="${wrist_3_inertia_iyz}"
-            izz="${wrist_3_inertia_izz}"
-        />
-      </inertial>
-    </link>
-    <!-- base_joint fixes base_link to the environment -->
-    <joint name="${tf_prefix}base_joint" type="fixed">
-      <xacro:insert_block name="origin" />
-      <parent link="${parent}" />
-      <child link="${tf_prefix}base_link" />
-    </joint>
+          <mesh filename="${forearm_collision_mesh}"/>
+        </geometry>
+      </collision>
+      <xacro:cylinder_inertial radius="${forearm_inertia_radius}" length="${forearm_inertia_length}"  mass="${forearm_mass}">
+        <origin xyz="${-0.5 * forearm_inertia_length} 0.0 ${elbow_offset}" rpy="0 ${pi/2} 0" />
+      </xacro:cylinder_inertial>
+    </link>
+    <link name="${prefix}wrist_1_link">
+      <visual>
+        <origin xyz="0 0 ${wrist_1_visual_offset}" rpy="${pi/2} 0 0"/>
+        <geometry>
+          <mesh filename="${wrist_1_visual_mesh}"/>
+        </geometry>
+        <material name="${wrist_1_visual_material_name}">
+          <color rgba="${wrist_1_visual_material_color}"/>
+        </material>
+      </visual>
+      <collision>
+        <origin xyz="0 0 ${wrist_1_visual_offset}" rpy="${pi/2} 0 0"/>
+        <geometry>
+          <mesh filename="${wrist_1_collision_mesh}"/>
+        </geometry>
+      </collision>
+      <xacro:cylinder_inertial radius="${wrist_1_inertia_radius}" length="${wrist_1_inertia_length}"  mass="${wrist_1_mass}">
+        <origin xyz="0 0 0" rpy="0 0 0" />
+      </xacro:cylinder_inertial>
+    </link>
+    <link name="${prefix}wrist_2_link">
+      <visual>
+        <origin xyz="0 0 ${wrist_2_visual_offset}" rpy="0 0 0"/>
+        <geometry>
+          <mesh filename="${wrist_2_visual_mesh}"/>
+        </geometry>
+        <material name="${wrist_2_visual_material_name}">
+          <color rgba="${wrist_2_visual_material_color}"/>
+        </material>
+      </visual>
+      <collision>
+        <origin xyz="0 0 ${wrist_2_visual_offset}" rpy="0 0 0"/>
+        <geometry>
+          <mesh filename="${wrist_2_collision_mesh}"/>
+        </geometry>
+      </collision>
+      <xacro:cylinder_inertial radius="${wrist_2_inertia_radius}" length="${wrist_2_inertia_length}"  mass="${wrist_2_mass}">
+        <origin xyz="0 0 0" rpy="0 0 0" />
+      </xacro:cylinder_inertial>
+    </link>
+    <link name="${prefix}wrist_3_link">
+      <visual>
+        <origin xyz="0 0 ${wrist_3_visual_offset}" rpy="${pi/2} 0 0"/>
+        <geometry>
+          <mesh filename="${wrist_3_visual_mesh}"/>
+        </geometry>
+        <material name="${wrist_3_visual_material_name}">
+          <color rgba="${wrist_3_visual_material_color}"/>
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