Commit message: tetsing with gripper and apporhc angle

File: ur_ws_new/src/universal_robot/urdf/ur_macro.xacro (robot description, xacro)
@@ -509,10 +509,10 @@
     <xacro:property name="hand_eye_zed_mini_left_camera_frame_new_lab_xyz" value="-0.123634 0.062070 0.084893"/>
     <xacro:property name="hand_eye_zed_mini_left_camera_frame_new_lab_rpy" value="-0.206146 0.001382 -1.835627"/>
-    <xacro:property name="hand_eye_zed_mini_left_camera_frame_new_outdoor_xyz" value="-0.123634 0.062070 0.084893"/>
-    <xacro:property name="hand_eye_zed_mini_left_camera_frame_new_outdoor_rpy" value="-0.206146 0.001382 -1.835627"/>
-    <xacro:property name="hand_eye_zed_mini_left_camera_frame_old_lab_xyz" value="-0.123634 0.062070 0.084893"/>
-    <xacro:property name="hand_eye_zed_mini_left_camera_frame_old_lab_rpy" value="-0.206146 0.001382 -1.835627"/>
-    <xacro:property name="hand_eye_zed_mini_left_camera_frame_old_outdoor_xyz" value="-0.123634 0.062070 0.084893"/>
-    <xacro:property name="hand_eye_zed_mini_left_camera_frame_old_outdoor_rpy" value="-0.206146 0.001382 -1.835627"/>
+    <xacro:property name="hand_eye_zed_mini_left_camera_frame_new_outdoor_xyz" value="-0.077883 -0.090478 0.078155"/>
+    <xacro:property name="hand_eye_zed_mini_left_camera_frame_new_outdoor_rpy" value="-0.202440 0.016049 -0.497189"/>
+    <xacro:property name="hand_eye_zed_mini_left_camera_frame_old_lab_xyz" value="-0.139864 -0.015226 0.081444"/>
+    <xacro:property name="hand_eye_zed_mini_left_camera_frame_old_lab_rpy" value="-0.193865 -0.018502 -1.265786"/>
+    <xacro:property name="hand_eye_zed_mini_left_camera_frame_old_outdoor_xyz" value="-0.078546 -0.089902 0.074421"/>
+    <xacro:property name="hand_eye_zed_mini_left_camera_frame_old_outdoor_rpy" value="-0.193188 -0.004251 -0.494148"/>
     <origin
       xyz="${hand_eye_zed_mini_left_camera_frame_new_lab_xyz if robot_profile == 'new' and environment == 'lab' else hand_eye_zed_mini_left_camera_frame_new_outdoor_xyz if robot_profile == 'new' else hand_eye_zed_mini_left_camera_frame_old_lab_xyz if environment == 'lab' else hand_eye_zed_mini_left_camera_frame_old_outdoor_xyz}"

Commit message: Calibrate gripper and improve hand-eye validation

File: ur_ws_new/src/universal_robot/urdf/ur_macro.xacro (robot description, xacro)
@@ -511,8 +511,8 @@
     <xacro:property name="hand_eye_zed_mini_left_camera_frame_new_outdoor_xyz" value="-0.077883 -0.090478 0.078155"/>
     <xacro:property name="hand_eye_zed_mini_left_camera_frame_new_outdoor_rpy" value="-0.202440 0.016049 -0.497189"/>
-    <xacro:property name="hand_eye_zed_mini_left_camera_frame_old_lab_xyz" value="-0.139864 -0.015226 0.081444"/>
-    <xacro:property name="hand_eye_zed_mini_left_camera_frame_old_lab_rpy" value="-0.193865 -0.018502 -1.265786"/>
-    <xacro:property name="hand_eye_zed_mini_left_camera_frame_old_outdoor_xyz" value="-0.078546 -0.089902 0.074421"/>
-    <xacro:property name="hand_eye_zed_mini_left_camera_frame_old_outdoor_rpy" value="-0.193188 -0.004251 -0.494148"/>
+    <xacro:property name="hand_eye_zed_mini_left_camera_frame_old_lab_xyz" value="-0.134119 -0.030555 0.088598"/>
+    <xacro:property name="hand_eye_zed_mini_left_camera_frame_old_lab_rpy" value="-0.232932 -0.069493 -1.113606"/>
+    <xacro:property name="hand_eye_zed_mini_left_camera_frame_old_outdoor_xyz" value="-0.087114 -0.084225 0.068128"/>
+    <xacro:property name="hand_eye_zed_mini_left_camera_frame_old_outdoor_rpy" value="-0.138898 0.016353 -0.605352"/>
     <origin
       xyz="${hand_eye_zed_mini_left_camera_frame_new_lab_xyz if robot_profile == 'new' and environment == 'lab' else hand_eye_zed_mini_left_camera_frame_new_outdoor_xyz if robot_profile == 'new' else hand_eye_zed_mini_left_camera_frame_old_lab_xyz if environment == 'lab' else hand_eye_zed_mini_left_camera_frame_old_outdoor_xyz}"

Commit message: Harden harvesting motion and add pollination workflow

File: ur_ws_new/src/universal_robot/urdf/ur_macro.xacro (robot description, xacro)
@@ -511,6 +511,6 @@
     <xacro:property name="hand_eye_zed_mini_left_camera_frame_new_outdoor_xyz" value="-0.077883 -0.090478 0.078155"/>
     <xacro:property name="hand_eye_zed_mini_left_camera_frame_new_outdoor_rpy" value="-0.202440 0.016049 -0.497189"/>
-    <xacro:property name="hand_eye_zed_mini_left_camera_frame_old_lab_xyz" value="-0.117001 -0.028902 0.072682"/>
-    <xacro:property name="hand_eye_zed_mini_left_camera_frame_old_lab_rpy" value="-0.114225 0.001975 -1.122874"/>
+    <xacro:property name="hand_eye_zed_mini_left_camera_frame_old_lab_xyz" value="-0.030796 -0.166455 0.004039"/>
+    <xacro:property name="hand_eye_zed_mini_left_camera_frame_old_lab_rpy" value="-0.014997 -0.001554 -0.024273"/>
     <xacro:property name="hand_eye_zed_mini_left_camera_frame_old_outdoor_xyz" value="-0.115138 -0.075365 0.080713"/>
     <xacro:property name="hand_eye_zed_mini_left_camera_frame_old_outdoor_rpy" value="-0.187840 -0.004377 -0.796829"/>

Commit message: Refresh the lab old ZED Mini hand-eye calibration
Re-calibrated 2026-09-30 from 20 samples with DANIILIDIS. Stationary-board translation error improved from 0.97mm median / 1.71mm p95 to 0.56mm median / 1.18mm p95, at the cost of slightly higher rotation error (0.065deg to 0.084deg median).

Updates the active profile, the top-level hand-eye YAML and the mirrored old_lab xyz/rpy properties in ur_macro.xacro so TF and the vision stack agree.

File: ur_ws_new/src/universal_robot/urdf/ur_macro.xacro (robot description, xacro)
@@ -511,6 +511,6 @@
     <xacro:property name="hand_eye_zed_mini_left_camera_frame_new_outdoor_xyz" value="-0.077883 -0.090478 0.078155"/>
     <xacro:property name="hand_eye_zed_mini_left_camera_frame_new_outdoor_rpy" value="-0.202440 0.016049 -0.497189"/>
-    <xacro:property name="hand_eye_zed_mini_left_camera_frame_old_lab_xyz" value="0.087639 -0.080624 0.074716"/>
-    <xacro:property name="hand_eye_zed_mini_left_camera_frame_old_lab_rpy" value="-0.108100 0.009920 1.053293"/>
+    <xacro:property name="hand_eye_zed_mini_left_camera_frame_old_lab_xyz" value="0.090454 -0.080254 0.073331"/>
+    <xacro:property name="hand_eye_zed_mini_left_camera_frame_old_lab_rpy" value="-0.113475 0.009291 1.050907"/>
     <xacro:property name="hand_eye_zed_mini_left_camera_frame_old_outdoor_xyz" value="-0.115138 -0.075365 0.080713"/>
     <xacro:property name="hand_eye_zed_mini_left_camera_frame_old_outdoor_rpy" value="-0.187840 -0.004377 -0.796829"/>

Commit message: Checkpoint timestamped demo recording and current grasp geometry

File: ur_ws_new/src/universal_robot/urdf/ur_macro.xacro (robot description, xacro)
@@ -530,5 +530,5 @@
   		<parent link="${tf_prefix}delto_base_link"/>
   		<child link="${tf_prefix}gripper_tip"/>
-		<origin xyz="0 0 0.115" rpy="0 0 0"/> <!-- Centered at the start of the fingertip pads -->
+		<origin xyz="0 0 0.145" rpy="0 0 0"/> <!-- Start of the fingertip pads, +30mm for the longer fingertips -->
 		</joint>
 <!-- Gripper tip frame -->

File: ur_ws_new/src/ur10e_curobo/ur10e_curobo/robot_assets/ur_description/ur10e_curobo.urdf (robot description, URDF)
Before this commit: robot ur10e, 31 links, 30 joints
Joints:
- joint gripper_link_to_tip: origin xyz=0 0 0.1 rpy=0 0.014 0.0 -> xyz=0 0 0.13 rpy=0 0.014 0.0
