Commit message: Recalibrate hand-eye transform for lab_old_zedx_mini_rgbd
Fresh eye-in-hand calibration for the old-robot/lab profile, propagated
to the URDF camera mount offset, the calibration record, and the active
camera profile YAML.

Co-Authored-By: Claude Sonnet 5 <noreply@anthropic.com>

File: ur_ws_new/src/universal_robot/urdf/ur_macro.xacro (robot description, xacro)
@@ -511,6 +511,6 @@
     <xacro:property name="hand_eye_zed_mini_left_camera_frame_new_outdoor_xyz" value="-0.077883 -0.090478 0.078155"/>
     <xacro:property name="hand_eye_zed_mini_left_camera_frame_new_outdoor_rpy" value="-0.202440 0.016049 -0.497189"/>
-    <xacro:property name="hand_eye_zed_mini_left_camera_frame_old_lab_xyz" value="-0.134119 -0.030555 0.088598"/>
-    <xacro:property name="hand_eye_zed_mini_left_camera_frame_old_lab_rpy" value="-0.232932 -0.069493 -1.113606"/>
+    <xacro:property name="hand_eye_zed_mini_left_camera_frame_old_lab_xyz" value="-0.136766 -0.014974 0.075378"/>
+    <xacro:property name="hand_eye_zed_mini_left_camera_frame_old_lab_rpy" value="-0.161942 -0.006961 -1.263528"/>
     <xacro:property name="hand_eye_zed_mini_left_camera_frame_old_outdoor_xyz" value="-0.087114 -0.084225 0.068128"/>
     <xacro:property name="hand_eye_zed_mini_left_camera_frame_old_outdoor_rpy" value="-0.138898 0.016353 -0.605352"/>

Commit message: Checkpoint outstanding workspace changes
Commits the remaining uncommitted working-tree changes as a restore point
before the multi-goal batching work. This is a checkpoint rather than a
single coherent change: it spans the vision node and visualization, the
Delto gripper driver and controller, grasp outcome classification, motion
and node plumbing, the RViz panel, launchers, URDF, and hand-eye/camera
calibration profiles.

Also drops two YOLO weight LFS pointers that are no longer referenced.

Not reviewed change-by-change; captured so the harvest-cycle work has a
clean point to fall back to.

Co-Authored-By: Claude Opus 5 <noreply@anthropic.com>

File: ur_ws_new/src/universal_robot/urdf/ur_macro.xacro (robot description, xacro)
@@ -511,8 +511,8 @@
     <xacro:property name="hand_eye_zed_mini_left_camera_frame_new_outdoor_xyz" value="-0.077883 -0.090478 0.078155"/>
     <xacro:property name="hand_eye_zed_mini_left_camera_frame_new_outdoor_rpy" value="-0.202440 0.016049 -0.497189"/>
-    <xacro:property name="hand_eye_zed_mini_left_camera_frame_old_lab_xyz" value="-0.136766 -0.014974 0.075378"/>
-    <xacro:property name="hand_eye_zed_mini_left_camera_frame_old_lab_rpy" value="-0.161942 -0.006961 -1.263528"/>
-    <xacro:property name="hand_eye_zed_mini_left_camera_frame_old_outdoor_xyz" value="-0.087114 -0.084225 0.068128"/>
-    <xacro:property name="hand_eye_zed_mini_left_camera_frame_old_outdoor_rpy" value="-0.138898 0.016353 -0.605352"/>
+    <xacro:property name="hand_eye_zed_mini_left_camera_frame_old_lab_xyz" value="-0.117001 -0.028902 0.072682"/>
+    <xacro:property name="hand_eye_zed_mini_left_camera_frame_old_lab_rpy" value="-0.114225 0.001975 -1.122874"/>
+    <xacro:property name="hand_eye_zed_mini_left_camera_frame_old_outdoor_xyz" value="-0.115038 -0.075192 0.082343"/>
+    <xacro:property name="hand_eye_zed_mini_left_camera_frame_old_outdoor_rpy" value="-0.183795 0.002590 -0.791661"/>
     <origin
       xyz="${hand_eye_zed_mini_left_camera_frame_new_lab_xyz if robot_profile == 'new' and environment == 'lab' else hand_eye_zed_mini_left_camera_frame_new_outdoor_xyz if robot_profile == 'new' else hand_eye_zed_mini_left_camera_frame_old_lab_xyz if environment == 'lab' else hand_eye_zed_mini_left_camera_frame_old_outdoor_xyz}"

Commit message: Stop writing 1970-stamped calibrations on a unit with no RTC battery
This Jetson has no battery-backed RTC, so an offline boot comes up at the
epoch. Two outdoor hand-eye calibrations were written that way -- 1970-01-01
03:09:10 and 03:24:20, i.e. 9 and 24 minutes past epoch -- leaving two
disagreeing profiles with no way to tell which was newer or which the robot
was actually flying.

Adopts the 26-sample run: mean error 2.57mm -> 2.14mm, translation max
3.05mm -> 2.15mm, at the cost of rotation p95 0.249deg -> 0.339deg. The
later epoch-03:24 run (rotation max 0.749deg, translation max 4.12mm) was
worse and is rejected. ur_macro.xacro carries the same values; cuRobo
rebuilds its URDF from the profile at startup, so these must stay in step.

The geometry in those files was never in question -- hand-eye only uses TF
within one session and the clock was stable, just wrong. Only provenance was
lost, so the profile now records why calibrated_at reads 1970.

A wrong clock is nearly harmless here: every node runs on this one machine
and shares it, so TF stays self-consistent. A clock that STEPS mid-session is
not -- every buffered transform goes decades stale at once, and
systemd-timesyncd always steps rather than slews. Fixed at the system level
with fake-hwclock (boot at last-known-good instead of the epoch) and chrony
"makestep 1 3" (step only in the first three updates, slew thereafter), so a
mid-harvest WiFi reconnect nudges instead of jumping.

unet.sh pulls the clock forward before any ROS node starts, and warns loudly
if it is still unset. hand_eye_calibration.py now refuses to write when the
year is implausible, rather than producing another untraceable file.

Co-Authored-By: Claude Opus 5 <noreply@anthropic.com>

File: ur_ws_new/src/universal_robot/urdf/ur_macro.xacro (robot description, xacro)
@@ -513,6 +513,6 @@
     <xacro:property name="hand_eye_zed_mini_left_camera_frame_old_lab_xyz" value="-0.117001 -0.028902 0.072682"/>
     <xacro:property name="hand_eye_zed_mini_left_camera_frame_old_lab_rpy" value="-0.114225 0.001975 -1.122874"/>
-    <xacro:property name="hand_eye_zed_mini_left_camera_frame_old_outdoor_xyz" value="-0.115038 -0.075192 0.082343"/>
-    <xacro:property name="hand_eye_zed_mini_left_camera_frame_old_outdoor_rpy" value="-0.183795 0.002590 -0.791661"/>
+    <xacro:property name="hand_eye_zed_mini_left_camera_frame_old_outdoor_xyz" value="-0.115138 -0.075365 0.080713"/>
+    <xacro:property name="hand_eye_zed_mini_left_camera_frame_old_outdoor_rpy" value="-0.187840 -0.004377 -0.796829"/>
     <origin
       xyz="${hand_eye_zed_mini_left_camera_frame_new_lab_xyz if robot_profile == 'new' and environment == 'lab' else hand_eye_zed_mini_left_camera_frame_new_outdoor_xyz if robot_profile == 'new' else hand_eye_zed_mini_left_camera_frame_old_lab_xyz if environment == 'lab' else hand_eye_zed_mini_left_camera_frame_old_outdoor_xyz}"

Commit message: Recalibrate hand-eye against a 9x14 40mm ChArUco board
The board parameters described a Calib.io 17x24 30mm/22mm board that is not
the one being held in front of the camera. Corrected to the 9x14 40mm/30mm
board actually in use, and the generated board image committed alongside so
the two cannot drift apart again.

Recalibrated on that board, 20 samples, DANIILIDIS. Residuals improved:
rotation median 0.159 -> 0.065deg, translation max 2.83 -> 2.07mm. Values
propagated to the lab camera profile and to ur_macro.xacro, which must stay
in step because cuRobo rebuilds its URDF from the profile at startup.

UNVERIFIED, and separated into its own commit so it can be reverted without
touching the motion work. The mount yaw moved ~62deg (rpy yaw -0.024 ->
+1.053 rad) against a translation that barely changed. That is either a real
remount or a solve that fits its own samples well while being wrong -- which
is exactly the failure 645268c79 added the acceptance test for, after a
calibration with 44 samples and all five methods within 1mm still shipped a
12.5deg yaw error. Low residuals do not rule it out.

Grasp success by day, small samples and not conclusive on its own:
13 Sep 67% (n=6), 14 Sep 54% (n=13), 16 Sep 27% (n=15, recalibrated 13:11),
17 Sep 50% (n=4). The grasp offsets in the previous commit were all fitted
on top of this calibration, so reverting one without the other will make
things worse rather than better.

Run the hand-eye acceptance test before trusting it.

Co-Authored-By: Claude Opus 5 <noreply@anthropic.com>

File: ur_ws_new/src/universal_robot/urdf/ur_macro.xacro (robot description, xacro)
@@ -511,6 +511,6 @@
     <xacro:property name="hand_eye_zed_mini_left_camera_frame_new_outdoor_xyz" value="-0.077883 -0.090478 0.078155"/>
     <xacro:property name="hand_eye_zed_mini_left_camera_frame_new_outdoor_rpy" value="-0.202440 0.016049 -0.497189"/>
-    <xacro:property name="hand_eye_zed_mini_left_camera_frame_old_lab_xyz" value="-0.030796 -0.166455 0.004039"/>
-    <xacro:property name="hand_eye_zed_mini_left_camera_frame_old_lab_rpy" value="-0.014997 -0.001554 -0.024273"/>
+    <xacro:property name="hand_eye_zed_mini_left_camera_frame_old_lab_xyz" value="0.087639 -0.080624 0.074716"/>
+    <xacro:property name="hand_eye_zed_mini_left_camera_frame_old_lab_rpy" value="-0.108100 0.009920 1.053293"/>
     <xacro:property name="hand_eye_zed_mini_left_camera_frame_old_outdoor_xyz" value="-0.115138 -0.075365 0.080713"/>
     <xacro:property name="hand_eye_zed_mini_left_camera_frame_old_outdoor_rpy" value="-0.187840 -0.004377 -0.796829"/>

Commit message: Speed up the harvest cycle and add local NuRec bag recording
- Faster gross motion: approach staging 0.8x, return HOME 0.8x, shorter
  approach endpoint settle and gripper close/settle waits (~16.1s -> ~14s
  per cycle measured).
- Batch harvest: test "go straight to next goal" in the background during
  DROP-OFF instead of standing still afterwards (~1s per goal after the
  first); queue only fruits seen in 2 of the last 3 vision frames.
- Episodes record level_final_z.
- NuRec: Start/Stop NuRec Bag buttons in the RViz Camera tab; the vision
  node records the stereo pair, TF and URDF to ~/nurec_data/bags locally.
- Outdoor hand-eye recalibration (2026-10-14), longer vision start delay,
  and ongoing demo capture/sequence, panel and planner work.

Co-Authored-By: Claude Opus 5.5 <noreply@anthropic.com>

File: ur_ws_new/src/universal_robot/urdf/ur_macro.xacro (robot description, xacro)
@@ -513,6 +513,6 @@
     <xacro:property name="hand_eye_zed_mini_left_camera_frame_old_lab_xyz" value="0.090454 -0.080254 0.073331"/>
     <xacro:property name="hand_eye_zed_mini_left_camera_frame_old_lab_rpy" value="-0.113475 0.009291 1.050907"/>
-    <xacro:property name="hand_eye_zed_mini_left_camera_frame_old_outdoor_xyz" value="-0.115138 -0.075365 0.080713"/>
-    <xacro:property name="hand_eye_zed_mini_left_camera_frame_old_outdoor_rpy" value="-0.187840 -0.004377 -0.796829"/>
+    <xacro:property name="hand_eye_zed_mini_left_camera_frame_old_outdoor_xyz" value="-0.023784 -0.117747 0.073093"/>
+    <xacro:property name="hand_eye_zed_mini_left_camera_frame_old_outdoor_rpy" value="-0.105417 0.010288 0.002149"/>
     <origin
       xyz="${hand_eye_zed_mini_left_camera_frame_new_lab_xyz if robot_profile == 'new' and environment == 'lab' else hand_eye_zed_mini_left_camera_frame_new_outdoor_xyz if robot_profile == 'new' else hand_eye_zed_mini_left_camera_frame_old_lab_xyz if environment == 'lab' else hand_eye_zed_mini_left_camera_frame_old_outdoor_xyz}"

File: ur_ws_new/src/ur10e_curobo/ur10e_curobo/robot_assets/ur_description/ur10e_curobo.urdf (robot description, URDF)
Before this commit: robot ur10e, 31 links, 30 joints
Joints:
- joint tool0_to_zed_mini_left_camera_frame: origin xyz=0.090454 -0.080254 0.073331 rpy=-0.113475 0.009291 1.050907 -> xyz=-0.023784 -0.117747 0.073093 rpy=-0.105417 0.010288 0.002149
