Commit message: newer deve bramnch 17eb

File: curobo/src/curobo/content/assets/robot/ur_description/ur10e_curobo.urdf (robot description, URDF)
Before this commit: robot ur10e, 30 links, 29 joints
Joints:
- joint tool0_to_zed2_left_camera_frame: origin xyz=-0.048 -0.156 -0.005 rpy=0 0 -0.174 -> xyz=-0.0326 -0.1167 0.0670 rpy=-0.146387 -0.085132 -0.050741

File: ur_ws_new/src/DELTO_ROS2/delto_description/urdf/delto_gripper_3f.xacro (robot description, xacro)
@@ -36,5 +36,5 @@
     <child  link="${prefix}delto_base_link"/>
     <!-- tweak these if your gripper origin isn’t at tool0 -->
-    <origin xyz="0 0 0.106" rpy="0 0 0"/>
+    <origin xyz="0 0 0.106" rpy="0 0 -0.40"/>
   </joint>
    <link name="${prefix}F1_01">

File: ur_ws_new/src/universal_robot/urdf/zedxminiv1/ur_macro.xacro (robot description, xacro)
@@ -451,7 +451,7 @@
     <link name="tool0_to_camera_mount_link">
   <visual>
-    <origin xyz="0.0 0.0 0.025" rpy="0 0 3.14159"/>
+    <origin xyz="0.0 0.0 -0.032" rpy="0 0 3.14159"/>
     <geometry>
-      <mesh filename="package://ur_description/meshes/ur10e/visual/zl_clamp_bo3.stl" scale="0.001 0.001 0.001"/>
+      <mesh filename="package://ur_description/meshes/ur10e/visual/top_zed_homut.stl" scale="0.001 0.001 0.001"/>
     </geometry>
     <material name="silver">
@@ -462,5 +462,5 @@
     <origin xyz="0.0 0.0 -0.032" rpy="0 0 3.14159"/>
     <geometry>
-      <mesh filename="package://ur_description/meshes/ur10e/visual/zl_clamp_bo3.stl" scale="0.001 0.001 0.001"/>
+      <mesh filename="package://ur_description/meshes/ur10e/visual/top_zed_homut.stl" scale="0.001 0.001 0.001"/>
     </geometry>
   </collision>
@@ -474,5 +474,5 @@
   <parent link="tool0"/>
   <child link="tool0_to_camera_mount_link"/>
-  <origin xyz="0 0 0" rpy="0 0 0"/>
+  <origin xyz="0 0 0" rpy="0 0 -0.174"/>
 </joint>
 <link name="zed2_left_camera_frame">
@@ -501,5 +501,5 @@
     <parent link="tool0"/>
     <child link="zed2_left_camera_frame"/>
-    <origin xyz="-0.0326 -0.1167 0.0670" rpy="-0.146387 -0.085132 -0.050741"/>   <!-- hand-eye calibrated (DANIILIDIS, 1.64mm error) -->
+    <origin xyz="-0.048 -0.156 -0.005" rpy="0 0 -0.174"/>   <!-- CHANGE -->
   </joint>
     <joint name="${tf_prefix}gripper_link_to_tip" type="fixed">

Commit message: fixed bugs and recalibrated

File: curobo/src/curobo/content/assets/robot/ur_description/ur10e_curobo.urdf (robot description, URDF)
Before this commit: robot ur10e, 30 links, 29 joints
Joints:
- joint tool0_to_zed2_left_camera_frame: origin xyz=-0.0326 -0.1167 0.0670 rpy=-0.146387 -0.085132 -0.050741 -> xyz=-0.026452 -0.116456 0.060776 rpy=-0.093175 0.004537 -0.010728

File: ur_ws_new/src/universal_robot/urdf/ur_macro.xacro (robot description, xacro)
@@ -501,5 +501,5 @@
     <parent link="tool0"/>
     <child link="zed2_left_camera_frame"/>
-    <origin xyz="-0.0326 -0.1167 0.0670" rpy="-0.146387 -0.085132 -0.050741"/>   <!-- hand-eye calibrated (DANIILIDIS, 1.64mm error) -->
+    <origin xyz="-0.026452 -0.116456 0.060776" rpy="-0.093175 0.004537 -0.010728"/>   <!-- hand-eye calibrated (DANIILIDIS, 1.79mm error) -->
   </joint>
     <joint name="${tf_prefix}gripper_link_to_tip" type="fixed">

Commit message: first commit for 2zed

File: curobo/src/curobo/content/assets/robot/ur_description/ur10e_curobo.urdf (robot description, URDF)
Before this commit: robot ur10e, 30 links, 29 joints
Links:
- added link zed_mini_left_camera_frame
Joints:
- added joint tool0_to_zed_mini_left_camera_frame: type fixed, parent tool0, child zed_mini_left_camera_frame, origin xyz=-0.000596 -0.146103 0.079483 rpy=-0.121254 -0.002856 -0.017912

File: ur_ws_new/src/universal_robot/urdf/ur_macro.xacro (robot description, xacro)
@@ -498,8 +498,16 @@
   </inertial>
 </link>
+  <!-- ZED X One Mono frame (derived: T_tool0_zedmini @ inv(T_CAM_ZEDMINI), 2026-04-15) — for RViz visualization -->
+  <link name="zed_mini_left_camera_frame"/>
+  <joint name="tool0_to_zed_mini_left_camera_frame" type="fixed">
+    <parent link="tool0"/>
+    <child link="zed_mini_left_camera_frame"/>
+    <origin xyz="-0.000596 -0.146103 0.079483" rpy="-0.121254 -0.002856 -0.017912"/>
+  </joint>
+  <!-- ZED X Mini frame (hand-eye calibrated, DANIILIDIS 1.79mm error) — CAM_FRAME, coords expressed in ZED Mini frame -->
   <joint name="tool0_to_zed2_left_camera_frame" type="fixed">
     <parent link="tool0"/>
     <child link="zed2_left_camera_frame"/>
-    <origin xyz="-0.026452 -0.116456 0.060776" rpy="-0.093175 0.004537 -0.010728"/>   <!-- hand-eye calibrated (DANIILIDIS, 1.79mm error) -->
+    <origin xyz="-0.026452 -0.116456 0.060776" rpy="-0.093175 0.004537 -0.010728"/>
   </joint>
     <joint name="${tf_prefix}gripper_link_to_tip" type="fixed">

Commit message: still in test

File: curobo/src/curobo/content/assets/robot/ur_description/ur10e_curobo.urdf (robot description, URDF)
Before this commit: robot ur10e, 31 links, 30 joints
Joints:
- joint tool0_to_zed2_left_camera_frame: origin xyz=-0.026452 -0.116456 0.060776 rpy=-0.093175 0.004537 -0.010728 -> xyz=0.029453 -0.148011 0.081938 rpy=-0.097892 -0.099072 0.218594

File: ur_ws_new/src/universal_robot/urdf/ur_macro.xacro (robot description, xacro)
@@ -505,9 +505,9 @@
     <origin xyz="-0.000596 -0.146103 0.079483" rpy="-0.121254 -0.002856 -0.017912"/>
   </joint>
-  <!-- ZED X Mini frame (hand-eye calibrated, DANIILIDIS 1.79mm error) — CAM_FRAME, coords expressed in ZED Mini frame -->
+  <!-- ZED X One frame (hand-eye calibrated, DANIILIDIS 2.45mm error, QHDPLUS, 2026-04-17) -->
   <joint name="tool0_to_zed2_left_camera_frame" type="fixed">
     <parent link="tool0"/>
     <child link="zed2_left_camera_frame"/>
-    <origin xyz="-0.026452 -0.116456 0.060776" rpy="-0.093175 0.004537 -0.010728"/>
+    <origin xyz="0.029453 -0.148011 0.081938" rpy="-0.097892 -0.099072 0.218594"/>
   </joint>
     <joint name="${tf_prefix}gripper_link_to_tip" type="fixed">

Commit message: tets

File: curobo/src/curobo/content/assets/robot/ur_description/ur10e_curobo.urdf (robot description, URDF)
Before this commit: robot ur10e, 31 links, 30 joints
Joints:
- joint tool0_to_zed2_left_camera_frame: origin xyz=0.029453 -0.148011 0.081938 rpy=-0.097892 -0.099072 0.218594 -> xyz=0.029402 -0.149589 0.082067 rpy=-0.086227 -0.104112 0.229781

File: ur_ws_new/src/universal_robot/urdf/ur_macro.xacro (robot description, xacro)
@@ -505,9 +505,9 @@
     <origin xyz="-0.000596 -0.146103 0.079483" rpy="-0.121254 -0.002856 -0.017912"/>
   </joint>
-  <!-- ZED X One frame (hand-eye calibrated, DANIILIDIS 2.45mm error, QHDPLUS, 2026-04-17) -->
+  <!-- ZED X One frame (hand-eye calibrated, DANIILIDIS 3.11mm error, QHDPLUS, 2026-04-19) -->
   <joint name="tool0_to_zed2_left_camera_frame" type="fixed">
     <parent link="tool0"/>
     <child link="zed2_left_camera_frame"/>
-    <origin xyz="0.029453 -0.148011 0.081938" rpy="-0.097892 -0.099072 0.218594"/>
+    <origin xyz="0.029402 -0.149589 0.082067" rpy="-0.086227 -0.104112 0.229781"/>
   </joint>
     <joint name="${tf_prefix}gripper_link_to_tip" type="fixed">

Commit message: tested and works

File: curobo/src/curobo/content/assets/robot/ur_description/ur10e_curobo.urdf (robot description, URDF)
Before this commit: robot ur10e, 31 links, 30 joints
Joints:
- joint tool0_to_zed2_left_camera_frame: origin xyz=0.029402 -0.149589 0.082067 rpy=-0.086227 -0.104112 0.229781 -> xyz=0.034102 -0.153032 0.079616 rpy=-0.172164 0.008484 0.204048

File: ur_ws_new/src/universal_robot/urdf/ur_macro.xacro (robot description, xacro)
@@ -509,5 +509,5 @@
     <parent link="tool0"/>
     <child link="zed2_left_camera_frame"/>
-    <origin xyz="0.029402 -0.149589 0.082067" rpy="-0.086227 -0.104112 0.229781"/>
+    <origin xyz="0.034102 -0.153032 0.079616" rpy="-0.172164 0.008484 0.204048"/><!-- hand-eye calibrated (DANIILIDIS, 2.05mm error, 32 samples, 2026-04-26) -->
   </joint>
     <joint name="${tf_prefix}gripper_link_to_tip" type="fixed">

File: ur_ws_new/src/ur10e_curobo/ur10e_curobo.urdf (robot description, URDF)
Before this commit: robot ur10e, 30 links, 29 joints
Joints:
- joint tool0_to_zed2_left_camera_frame: origin xyz=-0.06 -0.14 0.06 rpy=0 0 0 -> xyz=0.034102 -0.153032 0.079616 rpy=-0.172164 0.008484 0.204048

Commit message: workins may6

File: curobo/src/curobo/content/assets/robot/ur_description/ur10e_curobo.urdf (robot description, URDF)
Before this commit: robot ur10e, 31 links, 30 joints
Joints:
- joint tool0_to_zed2_left_camera_frame: origin xyz=0.034102 -0.153032 0.079616 rpy=-0.172164 0.008484 0.204048 -> xyz=0.042550 -0.150154 0.074587 rpy=-0.166668 0.013504 0.252667

File: ur_ws_new/src/universal_robot/urdf/ur_macro.xacro (robot description, xacro)
@@ -509,5 +509,5 @@
     <parent link="tool0"/>
     <child link="zed2_left_camera_frame"/>
-    <origin xyz="0.034102 -0.153032 0.079616" rpy="-0.172164 0.008484 0.204048"/><!-- hand-eye calibrated (DANIILIDIS, 2.05mm error, 32 samples, 2026-04-26) -->
+    <origin xyz="0.042550 -0.150154 0.074587" rpy="-0.166668 0.013504 0.252667"/><!-- hand-eye calibrated (DANIILIDIS, 4.02mm error, 36 samples, updated 2026-05-03 21:59:45) -->
   </joint>
     <joint name="${tf_prefix}gripper_link_to_tip" type="fixed">

Commit message: testng new tobot

File: curobo/src/curobo/content/assets/robot/ur_description/ur10e_curobo.urdf (robot description, URDF)
Before this commit: robot ur10e, 31 links, 30 joints
Joints:
- joint tool0_to_mount: origin xyz=0 0 -0.174 rpy=0 0 0 -> xyz=-0.008324 0.148998 0.040079 rpy=0 0 0
- joint tool0_to_zed2_left_camera_frame: origin xyz=0.042550 -0.150154 0.074587 rpy=-0.166668 0.013504 0.252667 -> xyz=-0.001111 0.153451 0.081263 rpy=-0.171298 -0.007406 -3.134152

File: ur_ws_new/src/universal_robot/urdf/ur.urdf.xacro (robot description, xacro)
@@ -8,4 +8,5 @@
    <!-- the default value should raise an error in case this was called without defining the type -->
    <xacro:arg name="ur_type" default="ur5x"/>
+   <xacro:arg name="robot_profile" default="new"/>
    <!-- parameters -->
    <xacro:arg name="tf_prefix" default="" />
@@ -80,4 +81,5 @@
    <xacro:ur_robot
      name="$(arg name)"
+     robot_profile="$(arg robot_profile)"
      tf_prefix="$(arg tf_prefix)"
      parent="world"

File: ur_ws_new/src/universal_robot/urdf/ur_macro.xacro (robot description, xacro)
@@ -47,4 +47,5 @@
   <xacro:macro name="ur_robot" params="
     name
+    robot_profile:=new
     tf_prefix
     parent
@@ -474,5 +475,7 @@
   <parent link="tool0"/>
   <child link="tool0_to_camera_mount_link"/>
-  <origin xyz="0 0 0" rpy="0 0 0"/>
+  <origin
+    xyz="${'-0.008324 0.148998 -0.016921' if robot_profile == 'new' else '0 0 0'}"
+    rpy="0 0 0"/>
 </joint>
 <link name="zed2_left_camera_frame">
@@ -509,5 +512,7 @@
     <parent link="tool0"/>
     <child link="zed2_left_camera_frame"/>
-    <origin xyz="0.042550 -0.150154 0.074587" rpy="-0.166668 0.013504 0.252667"/><!-- hand-eye calibrated (DANIILIDIS, 4.02mm error, 36 samples, updated 2026-05-03 21:59:45) -->
+    <origin
+      xyz="${'-0.001111 0.153451 0.081263' if robot_profile == 'new' else '0.042550 -0.150154 0.074587'}"
+      rpy="${'-0.171298 -0.007406 -3.134152' if robot_profile == 'new' else '-0.166668 0.013504 0.252667'}"/>
   </joint>
     <joint name="${tf_prefix}gripper_link_to_tip" type="fixed">

File: ur_ws_new/src/ur10e_curobo/ur10e_curobo.urdf (robot description, URDF)
Before this commit: robot ur10e, 30 links, 29 joints
Joints:
- joint tool0_to_mount: origin xyz=0 0 0 rpy=0 0 0 -> xyz=-0.116616 0.110078 -0.024749 rpy=0 0 0
- joint tool0_to_zed2_left_camera_frame: origin xyz=0.034102 -0.153032 0.079616 rpy=-0.172164 0.008484 0.204048 -> xyz=-0.001111 0.153451 0.081263 rpy=-0.171298 -0.007406 -3.134152
