Commit message: Checkpoint field grasp and perception improvements

File: curobo/src/curobo/content/assets/robot/ur_description/ur10e_curobo.urdf (robot description, URDF)
Before this commit: robot ur10e, 31 links, 30 joints
Links:
- link zed2_left_camera_frame: mass 0.4 -> None; geometry 
- link zed_mini_left_camera_frame: mass None -> 0.4; geometry collision mesh filename=package://ur_description/meshes/ur10e/visual/ZEDX_Mini.stl scale=0.001 0.001 0.001; visual mesh filename=package://ur_description/meshes/ur10e/visual/ZEDX_Mini.stl scale=0.001 0.001 0.001
Joints:
- removed joint tool0_to_mount
- added joint camera_to_mount: type fixed, parent zed_mini_left_camera_frame, child tool0_to_camera_mount_link, origin xyz=-0.000055 -0.008188 -0.039153 rpy=0 0 0
- joint tool0_to_zed_mini_left_camera_frame: origin xyz=-0.000596 -0.146103 0.079483 rpy=-0.121254 -0.002856 -0.017912 -> xyz=-0.123634 0.062070 0.084893 rpy=-0.206146 0.001382 -1.835627

File: ur_ws_new/src/universal_robot/urdf/ur.urdf.xacro (robot description, xacro)
@@ -9,4 +9,5 @@
    <xacro:arg name="ur_type" default="ur5x"/>
    <xacro:arg name="robot_profile" default="new"/>
+   <xacro:arg name="environment" default="outdoor"/>
    <!-- parameters -->
    <xacro:arg name="tf_prefix" default="" />
@@ -82,4 +83,5 @@
      name="$(arg name)"
      robot_profile="$(arg robot_profile)"
+     environment="$(arg environment)"
      tf_prefix="$(arg tf_prefix)"
      parent="world"

File: ur_ws_new/src/universal_robot/urdf/ur_macro.xacro (robot description, xacro)
@@ -48,4 +48,5 @@
     name
     robot_profile:=new
+    environment:=outdoor
     tf_prefix
     parent
@@ -472,12 +473,13 @@
   </inertial>
 </link>
-    <joint name="tool0_to_mount" type="fixed">
-  <parent link="tool0"/>
+    <joint name="camera_to_mount" type="fixed">
+  <parent link="zed_mini_left_camera_frame"/>
   <child link="tool0_to_camera_mount_link"/>
-  <origin
-    xyz="${'-0.008324 0.148998 -0.016921' if robot_profile == 'new' else '0 0 0'}"
-    rpy="0 0 0"/>
+  <!-- 40 mm below the camera along tool0 -Z, expressed in the camera frame. -->
+  <origin xyz="-0.000055 -0.008188 -0.039153" rpy="0 0 0"/>
 </joint>
-<link name="zed2_left_camera_frame">
+<link name="zed2_left_camera_frame"/>
+  <!-- ZED X Mini optical frame and RViz/collision geometry. -->
+  <link name="zed_mini_left_camera_frame">
   <visual>
     <origin xyz="0.007 0.01 -0.032" rpy="-3.142 0 0"/> <!-- hor ver -->
@@ -501,10 +503,19 @@
   </inertial>
 </link>
-  <!-- ZED X One Mono frame (derived: T_tool0_zedmini @ inv(T_CAM_ZEDMINI), 2026-04-15) — for RViz visualization -->
-  <link name="zed_mini_left_camera_frame"/>
   <joint name="tool0_to_zed_mini_left_camera_frame" type="fixed">
     <parent link="tool0"/>
     <child link="zed_mini_left_camera_frame"/>
-    <origin xyz="-0.000596 -0.146103 0.079483" rpy="-0.121254 -0.002856 -0.017912"/>
+    <!-- Each robot/environment pair owns an independent hand-eye transform. -->
+    <xacro:property name="hand_eye_zed_mini_left_camera_frame_new_lab_xyz" value="-0.123634 0.062070 0.084893"/>
+    <xacro:property name="hand_eye_zed_mini_left_camera_frame_new_lab_rpy" value="-0.206146 0.001382 -1.835627"/>
+    <xacro:property name="hand_eye_zed_mini_left_camera_frame_new_outdoor_xyz" value="-0.123634 0.062070 0.084893"/>
+    <xacro:property name="hand_eye_zed_mini_left_camera_frame_new_outdoor_rpy" value="-0.206146 0.001382 -1.835627"/>
+    <xacro:property name="hand_eye_zed_mini_left_camera_frame_old_lab_xyz" value="-0.123634 0.062070 0.084893"/>
+    <xacro:property name="hand_eye_zed_mini_left_camera_frame_old_lab_rpy" value="-0.206146 0.001382 -1.835627"/>
+    <xacro:property name="hand_eye_zed_mini_left_camera_frame_old_outdoor_xyz" value="-0.123634 0.062070 0.084893"/>
+    <xacro:property name="hand_eye_zed_mini_left_camera_frame_old_outdoor_rpy" value="-0.206146 0.001382 -1.835627"/>
+    <origin
+      xyz="${hand_eye_zed_mini_left_camera_frame_new_lab_xyz if robot_profile == 'new' and environment == 'lab' else hand_eye_zed_mini_left_camera_frame_new_outdoor_xyz if robot_profile == 'new' else hand_eye_zed_mini_left_camera_frame_old_lab_xyz if environment == 'lab' else hand_eye_zed_mini_left_camera_frame_old_outdoor_xyz}"
+      rpy="${hand_eye_zed_mini_left_camera_frame_new_lab_rpy if robot_profile == 'new' and environment == 'lab' else hand_eye_zed_mini_left_camera_frame_new_outdoor_rpy if robot_profile == 'new' else hand_eye_zed_mini_left_camera_frame_old_lab_rpy if environment == 'lab' else hand_eye_zed_mini_left_camera_frame_old_outdoor_rpy}"/>
   </joint>
   <!-- ZED X One frame (hand-eye calibrated, DANIILIDIS 3.11mm error, QHDPLUS, 2026-04-19) -->
