Commit message: Align gripper grasp frame and retune final grasp defaults

File: ur_ws_new/src/DELTO_ROS2/delto_description/urdf/delto_gripper_3f.xacro (robot description, xacro)
@@ -36,5 +36,7 @@
     <child  link="${prefix}delto_base_link"/>
     <!-- tweak these if your gripper origin isn’t at tool0 -->
-    <origin xyz="0 0 0.106" rpy="0 0 -0.40"/>
+    <!-- Match the physical mounting: isolated finger below the upper pair.
+         This adds a 90-degree clockwise visual roll about the tool axis. -->
+    <origin xyz="0 0 0.106" rpy="0 0 -1.97079632679"/>
   </joint>
    <link name="${prefix}F1_01">

File: ur_ws_new/src/universal_robot/urdf/ur_macro.xacro (robot description, xacro)
@@ -530,5 +530,5 @@
   		<parent link="${tf_prefix}delto_base_link"/>
   		<child link="${tf_prefix}gripper_tip"/>
-  		<origin xyz="0 0.014 0.09" rpy="0 0 0"/> <!-- Match the box length -->
+		<origin xyz="0 0 0.115" rpy="0 0 0"/> <!-- Centered at the start of the fingertip pads -->
 		</joint>
 <!-- Gripper tip frame -->

File: ur_ws_new/src/universal_robot/urdf/zed2iurdf/ur_macro.xacro (robot description, xacro)
@@ -506,5 +506,5 @@
   		<parent link="${tf_prefix}delto_base_link"/>
   		<child link="${tf_prefix}gripper_tip"/>
-  		<origin xyz="0 0 0.1" rpy="0 0 0"/> <!-- Match the box length -->
+		<origin xyz="0 0 0.115" rpy="0 0 0"/> <!-- Centered at the start of the fingertip pads -->
 		</joint>
 <!-- Gripper tip frame -->

File: ur_ws_new/src/universal_robot/urdf/zedxminiv1/ur_macro.xacro (robot description, xacro)
@@ -506,5 +506,5 @@
   		<parent link="${tf_prefix}delto_base_link"/>
   		<child link="${tf_prefix}gripper_tip"/>
-  		<origin xyz="0 0.014 0.09" rpy="0 0 0"/> <!-- Match the box length -->
+		<origin xyz="0 0 0.115" rpy="0 0 0"/> <!-- Centered at the start of the fingertip pads -->
 		</joint>
 <!-- Gripper tip frame -->

File: ur_ws_new/src/ur10e_curobo/ur10e_curobo.urdf (robot description, URDF)
Before this commit: robot ur10e, 30 links, 29 joints
Joints:
- joint gripper_link_to_tip: origin xyz=0 0 0.1 rpy=0 0 0 -> xyz=0 0 0.115 rpy=0 0 0
