Commit message: Carry the current hand-eye into the cuRobo source URDF
The baked-in tool0 -> zed_mini_left_camera_frame origin held the NEW robot's
lab mount, 257mm from this robot's. hand_eye_calibration.yaml, the camera
profile and ur_macro.xacro were all updated by the 2026-09-30 calibration
run; this file was not, because the calibration writer does not touch it.

Harmless most of the time and that is the problem. motion_executor rewrites
this origin per camera profile at startup, but only when the profile carries
BOTH translation and rpy:

    if required_translation and required_rpy:   -> patch
    else                                        -> warn, use the source as-is

The else branch is not hypothetical. Every Isaac Jetson launch before
90f8fcd6d took it, because that path set no UR10E_CAMERA_PROFILE and fell
back to zed_one_rgb_zedx_mini_depth.yaml, which carries only a seed. Those
runs planned with another robot's camera mount, and the only clue was one
warning line.

Now the fallback is this robot's actual calibration, so taking that branch
degrades to slightly stale rather than badly wrong.

  xyz  -0.123634  0.062070  0.084893  ->  0.090454 -0.080254  0.073331
  rpy  -0.206146  0.001382 -1.835627  -> -0.113475  0.009291  1.050907

Values are the matrix translation and the quaternion of
hand_eye_calibration.yaml (DANIILIDIS, 20 samples, 2026-09-30 12:41:34),
converted to rpy and verified to agree within 0.0004mm and 0.0000deg.

tool0_to_zed2_left_camera_frame is deliberately untouched: different camera,
its own June calibration, and no current solve exists for it.

Checked the generator still works on the edited file -- its regex finds the
joint and exactly one origin tag, which is what it requires before patching.
A second origin, or none, would make it error and silently fall back. Suite
80/80.

Co-Authored-By: Claude Opus 5 <noreply@anthropic.com>

File: ur_ws_new/src/ur10e_curobo/ur10e_curobo/robot_assets/ur_description/ur10e_curobo.urdf (robot description, URDF)
Before this commit: robot ur10e, 31 links, 30 joints
Joints:
- joint tool0_to_zed_mini_left_camera_frame: origin xyz=-0.123634 0.062070 0.084893 rpy=-0.206146 0.001382 -1.835627 -> xyz=0.090454 -0.080254 0.073331 rpy=-0.113475 0.009291 1.050907
